Commit message: Adding some controllers for Robotics exam :)

File: src/modelo_robot/urdf/robot.urdf.xacro (robot description, xacro)
@@ -5,4 +5,6 @@
     <xacro:include filename="ensamblaje.xacro" />
     <xacro:include filename="lidar.xacro" />
-    <xacro:include filename="ros2_control.xacro"/>
+    <!--xacro:include filename="ros2_control.xacro"/-->
+    <!--xacro:include filename="position_control.xacro"/-->
+    <xacro:include filename="trajectory_controller.xacro"/>
 </robot>

File: src/modelo_robot/urdf/trajectory_controller.xacro (robot description, xacro)
@@ -7,6 +7,6 @@
       <joint name="rueda_izq_delantera_joint">
           <command_interface name="position">
-            <param name="min">-100000 </param>
-            <param name="max">100000 </param>
+            <param name="min">-10 </param>
+            <param name="max">10 </param>
           </command_interface>
           <state_interface name="position"/>
@@ -14,28 +14,4 @@
         </joint>
         <joint name="rueda_der_delantera_joint">
-          <command_interface name="position">
-            <param name="min">-100000 </param>
-            <param name="max">100000 </param>
-          </command_interface>
-          <state_interface name="position"/>
-          <state_interface name="velocity"/>
-        </joint>
-        <joint name="rueda_izq_trasera_joint">
-          <command_interface name="position">
-            <param name="min">-100000 </param>
-            <param name="max">100000 </param>
-          </command_interface>
-          <state_interface name="position"/>
-          <state_interface name="velocity"/>
-        </joint>
-        <joint name="rueda_der_trasera_joint">
-          <command_interface name="position">
-            <param name="min">-100000 </param>
-            <param name="max">100000 </param>
-          </command_interface>
-          <state_interface name="position"/>
-          <state_interface name="velocity"/>
-        </joint>
-        <joint name="aspersor_joint">
           <command_interface name="position">
             <param name="min">-10 </param>
@@ -45,8 +21,32 @@
           <state_interface name="velocity"/>
         </joint>
+        <joint name="rueda_izq_trasera_joint">
+          <command_interface name="position">
+            <param name="min">-10 </param>
+            <param name="max">10 </param>
+          </command_interface>
+          <state_interface name="position"/>
+          <state_interface name="velocity"/>
+        </joint>
+        <joint name="rueda_der_trasera_joint">
+          <command_interface name="position">
+            <param name="min">-10 </param>
+            <param name="max">10 </param>
+          </command_interface>
+          <state_interface name="position"/>
+          <state_interface name="velocity"/>
+        </joint>
+        <joint name="aspersor_joint">
+          <command_interface name="position">
+            <param name="min">-1.57 </param>
+            <param name="max">1.57 </param>
+          </command_interface>
+          <state_interface name="position"/>
+          <state_interface name="velocity"/>
+        </joint>
     </ros2_control>
     <gazebo>
       <plugin filename="libgazebo_ros2_control.so" name="gazebo_ros2_control">
-        <parameters>/home/andres/agrobot/src/modelo_robot/config/pos_controllers.yaml</parameters>
+        <parameters>/home/andres/agrobot/src/modelo_robot/config/trajectory_controller.yaml</parameters>
       </plugin>
     </gazebo>
