Commit message: Changing urdf to xacros for better organization and lidar functioning correctly

File: src/modelo_robot/urdf/ensamblaje.xacro (robot description, xacro)
@@ -3,7 +3,22 @@
      Commit Version: 1.6.0-4-g7f85cfe  Build Version: 1.6.7995.38578
      For more information, please see http://wiki.ros.org/sw_urdf_exporter -->
-<robot name="robot">
-  <link
-    name="base_link">
+<robot xmlns:xacro="http://www.ros.org/wiki/xacro" >
+  <link name="base_link">
+    </link>
+    <!-- BASE_FOOTPRINT LINK -->
+    <joint name="base_footprint_joint" type="fixed">
+        <parent link="base_link"/>
+        <child link="base_footprint"/>
+        <origin xyz="0 0 0" rpy="0 0 0"/>
+    </joint>
+    <link name="base_footprint">
+    </link>
+  <joint name="chassis_joint" type="fixed">
+        <parent link="base_link"/>
+        <child link="chassis"/>
+        <origin xyz="0 0 0"/>
+    </joint>
+  <link
+    name="chassis">
     <inertial>
       <origin
@@ -44,9 +59,5 @@
     </collision>
   </link>
-  <gazebo reference="base_link">
-    <mu1>0.001</mu1>
-    <mu2>0.001</mu2>
-    <kp>1000000</kp>
-    <kd>1</kd>
+  <gazebo reference="chassis">
     <material>Gazebo/Yellow</material>
   </gazebo>
@@ -366,83 +377,13 @@
       link="apersor_link" />
     <axis
-      xyz="0 0 1" />
-    <limit
-      lower="0"
-      upper="0"
-      effort="0"
-      velocity="100" />
-    <dynamics
-      damping="0.1"
-      friction="0.1" />
-  </joint>
-  <link name="lindar_link">
-    <inertial>
-      <origin xyz="-2.7756E-17 0.01 0" rpy="0 0 0" />
-      <mass value="0.066366" />
-      <inertia
-        ixx="1.9737E-05"
-        ixy="-2.8234E-22"
-        ixz="-2.8411E-21"
-        iyy="3.505E-05"
-        iyz="-1.4117E-22"
-        izz="1.9737E-05" />
-    </inertial>
-    <visual>
-      <origin xyz="0 0 0" rpy="0 0 0" />
-      <geometry>
-        <mesh filename="package://modelo_robot/meshes/lindar_link.STL" />
-      </geometry>
-      <material name="">
-        <color rgba="0.79216 0.81961 0.93333 1" />
-      </material>
-    </visual>
-    <collision>
-      <origin xyz="0 0 0" rpy="0 0 0" />
-      <geometry>
-        <mesh filename="package://modelo_robot/meshes/lindar_link.STL" />
-      </geometry>
-    </collision>
-  </link>
-  <gazebo reference="lindar_link">
-    <material>Gazebo/Blue</material>
-  </gazebo>
-  <joint name="lidar_frame" type="fixed">
-    <origin xyz="0.031539 -0.0015685 0.17" rpy="1.5708 0 3.1416" />
-    <parent link="base_link" />
-    <child link="lindar_link" />
-    <axis xyz="0 0 0" />
-  </joint>
-    <!-- Gazebo Plugins -->
-    <gazebo>
-        <plugin name="diff_drive" filename="libgazebo_ros_diff_drive.so">
-            <update_rate>100</update_rate>
-            <num_wheel_pairs>2</num_wheel_pairs>
-            <!-- Wheel Information -->
-            <left_joint>rueda_izq_trasera_joint</left_joint>
-            <left_joint>rueda_izq_delantera_joint</left_joint>
-            <right_joint>rueda_der_trasera_joint</right_joint>
-            <right_joint>rueda_der_delantera_joint</right_joint>
-            <wheel_separation>0.20</wheel_separation>
-            <wheel_radius>0.122</wheel_radius>
-            <!-- Limits -->
-            <max_linear_acceleration>5</max_linear_acceleration>
-            <min_linear_acceleration>-5</min_linear_acceleration>
-            <max_angular_acceleration>4</max_angular_acceleration>
-            <min_angular_acceleration>-4</min_angular_acceleration>
-            <!-- Receive velocity commands on this ROS topic -->
-            <command_topic>cmd_vel</command_topic>
-            <!-- output -->
-            <!-- When false, publish no wheel odometry data to a ROS topic -->
-            <publish_odom>true</publish_odom>
-            <!-- When true, publish coordinate transform from odom to base_footprint -->
-            <!-- I usually use the robot_localization package to publish this transform -->
-            <publish_odom_tf>true</publish_odom_tf>
-            <!-- When true, publish coordinate transform from base_link to the wheels -->
-            <!-- The robot_state_publisher package is often used to publish this transform -->
-            <publish_wheel_tf>true</publish_wheel_tf>
-            <odometry_topic>odom</odometry_topic>
-            <odometry_frame>odom_link</odometry_frame>
-            <robot_base_frame>base_link</robot_base_frame>
-        </plugin>
-    </gazebo>
+      xyz="0 1 0" />
+    <limit
+      lower="-1.5707"
+      upper="1.5707"
+      effort="5"
+      velocity="1" />
+    <dynamics
+      damping="0.1"
+      friction="0.1" />
+  </joint>
 </robot>

Commit message: Adding diff_controller in xacro

File: src/modelo_robot/urdf/ensamblaje.xacro (robot description, xacro)
@@ -373,5 +373,5 @@
       rpy="1.5708 0 3.1416" />
     <parent
-      link="base_link" />
+      link="chassis" />
     <child
       link="apersor_link" />

File: src/modelo_robot/urdf/lidar.xacro (robot description, xacro)
@@ -27,5 +27,5 @@
   <joint name="lidar_frame" type="fixed">
     <origin xyz="0.031539 -0.0015685 0.17" rpy="0 0 0" />
-    <parent link="chassis" />
+    <parent link="base_link" />
     <child link="lindar_link" />
     <axis xyz="0 0 0" />

File: src/modelo_robot/urdf/robot.urdf.xacro (robot description, xacro)
@@ -1,6 +1,8 @@
 <?xml version="1.0"?>
 <robot xmlns:xacro="http://www.ros.org/wiki/xacro"  name="robot">
+    <xacro:arg name="use_ros2_control" default="true"/>
+    <xacro:arg name="sim_mode" default="true"/>
     <xacro:include filename="ensamblaje.xacro" />
     <xacro:include filename="lidar.xacro" />
-    <xacro:include filename="gazebo_control.xacro" />
+    <xacro:include filename="ros2_control.xacro" />
 </robot>

Commit message: Fixing controllers and tf's in rviz

File: src/modelo_robot/urdf/ensamblaje.xacro (robot description, xacro)
@@ -4,21 +4,6 @@
      For more information, please see http://wiki.ros.org/sw_urdf_exporter -->
 <robot xmlns:xacro="http://www.ros.org/wiki/xacro" >
-  <link name="base_link">
-    </link>
-    <!-- BASE_FOOTPRINT LINK -->
-    <joint name="base_footprint_joint" type="fixed">
-        <parent link="base_link"/>
-        <child link="base_footprint"/>
-        <origin xyz="0 0 0" rpy="0 0 0"/>
-    </joint>
-    <link name="base_footprint">
-    </link>
-  <joint name="chassis_joint" type="fixed">
-        <parent link="base_link"/>
-        <child link="chassis"/>
-        <origin xyz="0 0 0"/>
-    </joint>
-  <link
-    name="chassis">
+  <link
+    name="base_link">
     <inertial>
       <origin
@@ -59,5 +44,5 @@
     </collision>
   </link>
-  <gazebo reference="chassis">
+  <gazebo reference="base_link">
     <material>Gazebo/Yellow</material>
   </gazebo>
@@ -122,8 +107,4 @@
   </joint>
   <gazebo reference="rueda_izq_delantera_link">
-    <mu1>0.001</mu1>
-    <mu2>0.001</mu2>
-    <kp>1000000</kp>
-    <kd>1</kd>
     <material>Gazebo/Gray</material>
   </gazebo>
@@ -169,8 +150,4 @@
   </link>
   <gazebo reference="rueda_izq_trasera_link">
-    <mu1>0.001</mu1>
-    <mu2>0.001</mu2>
-    <kp>1000000</kp>
-    <kd>1</kd>
     <material>Gazebo/Gray</material>
   </gazebo>
@@ -235,8 +212,4 @@
   </link>
   <gazebo reference="rueda_der_delantera_link">
-    <mu1>0.001</mu1>
-    <mu2>0.001</mu2>
-    <kp>1000000</kp>
-    <kd>1</kd>
     <material>Gazebo/Gray</material>
   </gazebo>
@@ -301,8 +274,4 @@
   </link>
   <gazebo reference="rueda_der_trasera_link">
-    <mu1>0.001</mu1>
-    <mu2>0.001</mu2>
-    <kp>1000000</kp>
-    <kd>1</kd>
     <material>Gazebo/Gray</material>
   </gazebo>
@@ -327,5 +296,5 @@
   </joint>
   <link
-    name="apersor_link">
+    name="aspersor_link">
     <inertial>
       <origin
@@ -348,5 +317,5 @@
       <geometry>
         <mesh
-          filename="package://modelo_robot/meshes/apersor_link.STL" />
+          filename="package://modelo_robot/meshes/aspersor_link.STL" />
       </geometry>
       <material
@@ -362,8 +331,11 @@
       <geometry>
         <mesh
-          filename="package://modelo_robot/meshes/apersor_link.STL" />
-      </geometry>
-    </collision>
-  </link>
+          filename="package://modelo_robot/meshes/aspersor_link.STL" />
+      </geometry>
+    </collision>
+  </link>
+  <gazebo reference="aspersor_link">
+    <material>Gazebo/Blue</material>
+  </gazebo>
   <joint
     name="aspersor_joint"
@@ -373,7 +345,7 @@
       rpy="1.5708 0 3.1416" />
     <parent
-      link="chassis" />
-    <child
-      link="apersor_link" />
+      link="base_link" />
+    <child
+      link="aspersor_link" />
     <axis
       xyz="0 1 0" />
@@ -383,7 +355,4 @@
       effort="5"
       velocity="1" />
-    <dynamics
-      damping="0.1"
-      friction="0.1" />
   </joint>
 </robot>

File: src/modelo_robot/urdf/lidar.xacro (robot description, xacro)
@@ -2,10 +2,12 @@
 <robot xmlns:xacro="http://www.ros.org/wiki/xacro" >
    <xacro:include filename="inertial_macros.xacro"/>
-  <link name="lindar_link">
+  <link name="laser_frame">
           <visual>
               <geometry>
                   <cylinder radius="0.03" length="0.02"/>
               </geometry>
-              <material name="black"/>
+              <material name="black">
+                    <color rgba="0 0 0 1"/>
+                </material>
           </visual>
           <visual>
@@ -14,5 +16,7 @@
                   <cylinder radius="0.01" length="0.1"/>
               </geometry>
-              <material name="black"/>
+              <material name="black">
+                    <color rgba="0 0 0 1"/>
+                </material>
           </visual>
           <collision>
@@ -25,11 +29,11 @@
           </xacro:inertial_cylinder>
       </link>
-  <joint name="lidar_frame" type="fixed">
+  <joint name="laser_joint" type="fixed">
     <origin xyz="0.031539 -0.0015685 0.17" rpy="0 0 0" />
     <parent link="base_link" />
-    <child link="lindar_link" />
+    <child link="laser_frame" />
     <axis xyz="0 0 0" />
   </joint>
-  <gazebo reference="lindar_link">
+  <gazebo reference="laser_frame">
         <material>Gazebo/Blue</material>
         <sensor name="laser" type="ray">

File: src/modelo_robot/urdf/robot.urdf.xacro (robot description, xacro)
@@ -5,4 +5,4 @@
     <xacro:include filename="ensamblaje.xacro" />
     <xacro:include filename="lidar.xacro" />
-    <xacro:include filename="ros2_control.xacro" />
+    <xacro:include filename="ros2_control.xacro"/>
 </robot>

File: src/modelo_robot/urdf/ros2_control.xacro (robot description, xacro)
@@ -38,4 +38,12 @@
           <state_interface name="position"/>
         </joint>
+        <joint name="aspersor_joint">
+          <command_interface name="velocity">
+            <param name="min">-10 </param>
+            <param name="max">10 </param>
+          </command_interface>
+          <state_interface name="velocity"/>
+          <state_interface name="position"/>
+        </joint>
     </ros2_control>
     <gazebo>

Commit message: Adding changes

File: src/modelo_robot/urdf/ensamblaje.xacro (robot description, xacro)
@@ -4,6 +4,24 @@
      For more information, please see http://wiki.ros.org/sw_urdf_exporter -->
 <robot xmlns:xacro="http://www.ros.org/wiki/xacro" >
-  <link
-    name="base_link">
+<xacro:include filename="inertial_macros.xacro"/>
+<!-- BASE LINK -->
+    <link name="base_link">
+    </link>
+    <!-- BASE_FOOTPRINT LINK -->
+<joint name="base_footprint_joint" type="fixed">
+        <parent link="base_link"/>
+        <child link="base_footprint"/>
+        <origin xyz="0 0 0" rpy="0 0 0"/>
+    </joint>
+    <link name="base_footprint">
+    </link>
+    <!-- CHASSIS LINK -->
+    <joint name="chassis_joint" type="fixed">
+        <parent link="base_link"/>
+        <child link="chassis"/>
+        <origin xyz="0 0 0"/>
+    </joint>
+  <link
+    name="chassis">
     <inertial>
       <origin
@@ -44,5 +62,5 @@
     </collision>
   </link>
-  <gazebo reference="base_link">
+  <gazebo reference="chassis">
     <material>Gazebo/Yellow</material>
   </gazebo>

File: src/modelo_robot/urdf/lidar.xacro (robot description, xacro)
@@ -1,5 +1,9 @@
 <?xml version="1.0"?>
 <robot xmlns:xacro="http://www.ros.org/wiki/xacro" >
-   <xacro:include filename="inertial_macros.xacro"/>
+    <joint name="laser_joint" type="fixed">
+        <origin xyz="0.031539 -0.0015685 0.20" rpy="0 0 0" />
+        <parent link="chassis" />
+        <child link="laser_frame" />
+    </joint>
   <link name="laser_frame">
           <visual>
@@ -22,5 +26,5 @@
           <collision>
               <geometry>
-                  <cylinder radius="0.05" length="0.04"/>
+                  <cylinder radius="0.03" length="0.02"/>
               </geometry>
           </collision>
@@ -29,10 +33,4 @@
           </xacro:inertial_cylinder>
       </link>
-  <joint name="laser_joint" type="fixed">
-    <origin xyz="0.031539 -0.0015685 0.17" rpy="0 0 0" />
-    <parent link="base_link" />
-    <child link="laser_frame" />
-    <axis xyz="0 0 0" />
-  </joint>
   <gazebo reference="laser_frame">
         <material>Gazebo/Blue</material>

File: src/modelo_robot/urdf/robot2.urdf.xacro (robot description, xacro)
@@ -3,7 +3,7 @@
     <xacro:arg name="use_ros2_control" default="true"/>
     <xacro:arg name="sim_mode" default="true"/>
-    <xacro:include filename="ensamblaje.xacro" />
-    <xacro:include filename="lidar.xacro" />
-    <xacro:include filename="ros2_control.xacro"/>
+    <xacro:include filename="robot2_core.xacro" />
+    <xacro:include filename="lidar2.xacro" />
+    <xacro:include filename="ros_control_robot2.xacro"/>
     <!--xacro:include filename="control_arduino.xacro"/-->
 </robot>

File: src/modelo_robot/urdf/robot_real.urdf.xacro (robot description, xacro)
@@ -2,8 +2,7 @@
 <robot xmlns:xacro="http://www.ros.org/wiki/xacro"  name="robot">
     <xacro:arg name="use_ros2_control" default="true"/>
-    <xacro:arg name="sim_mode" default="true"/>
+    <xacro:arg name="sim_mode" default="false"/>
     <xacro:include filename="ensamblaje.xacro" />
     <xacro:include filename="lidar.xacro" />
-    <xacro:include filename="ros2_control.xacro"/>
-    <!--xacro:include filename="control_arduino.xacro"/-->
+    <xacro:include filename="control_arduino.xacro"/>
 </robot>
